Commit message: Minor tweaks to fix warnings

File: vector_common/vector_description/urdf/accessories.urdf.xacro (robot description, xacro)
@@ -26,5 +26,5 @@
     <xacro:include filename="$(find vector_description)/urdf/sensors/pgr_flea3.urdf.xacro"/>
     <xacro:include filename="$(find vector_description)/urdf/sensors/pan_tilt_kinect_one.urdf.xacro" />
-    <property name="M_PI" value="3.14159"/>
+    <xacro:property name="M_PI" value="3.14159"/>
     <xacro:macro name="vector_accessories">
         <link name="sic_imu_frame"/>

File: vector_common/vector_description/urdf/manipulation/jaco/jaco.transmission.xacro (robot description, xacro)
@@ -1,4 +1,4 @@
 <?xml version="1.0"?>
-<robot xmlns:xacro="http://www.ros.org/wiki/xacro">
+<robot xmlns:xacro="http://ros.org/wiki/xacro">
   <xacro:macro name="jaco_arm_transmission" params="prefix">
     <transmission name="${prefix}shoulder_pan_trans">

File: vector_common/vector_description/urdf/manipulation/jaco/jaco.urdf.xacro (robot description, xacro)
@@ -21,15 +21,15 @@
 ARISING IN ANY WAY OUT OF THE USE OF THIS SOFTWARE, EVEN IF ADVISED OF THE POSSIBILITY OF SUCH DAMAGE.
 -->
-<robot name="jaco_robot" xmlns:xacro="http://www.ros.org/wiki/xacro">
+<robot name="jaco_robot" xmlns:xacro="http://ros.org/wiki/xacro">
     <xacro:include filename="$(find vector_description)/urdf/manipulation/jaco/jaco.transmission.xacro" />
-    <property name="M_PI" value="3.14159265"/>
+    <xacro:property name="M_PI" value="3.14159265"/>
     <!-- Inertia parameters -->
-    <property name="base_mass" value="0.752103" />
-    <property name="shoulder_mass" value="0.839784" />
-    <property name="upper_arm_mass" value="0.968862" />
-    <property name="forearm_mass" value="0.709960" />
-    <property name="wrist_1_mass" value="0.441232" />
-    <property name="wrist_2_mass" value="0.441232" />
-    <property name="wrist_3_mass" value="0.363290" />
+    <xacro:property name="base_mass" value="0.752103" />
+    <xacro:property name="shoulder_mass" value="0.839784" />
+    <xacro:property name="upper_arm_mass" value="0.968862" />
+    <xacro:property name="forearm_mass" value="0.709960" />
+    <xacro:property name="wrist_1_mass" value="0.441232" />
+    <xacro:property name="wrist_2_mass" value="0.441232" />
+    <xacro:property name="wrist_3_mass" value="0.363290" />
     <xacro:macro name="jaco_robot" params="prefix parent *origin">
         <joint name="${prefix}kinova_joint" type="fixed">

File: vector_common/vector_description/urdf/manipulation/robotiq/robotiq_85_gripper.transmission.xacro (robot description, xacro)
@@ -1,4 +1,4 @@
 <?xml version="1.0"?>
-<robot xmlns:xacro="http://www.ros.org/wiki/xacro">
+<robot xmlns:xacro="http://ros.org/wiki/xacro">
   <xacro:macro name="robotiq_85_gripper_transmission" params="prefix">
         <transmission name="${prefix}robotiq_85_left_knuckle_trans">

File: vector_common/vector_description/urdf/manipulation/robotiq/robotiq_85_gripper.urdf.xacro (robot description, xacro)
@@ -2,5 +2,5 @@
 <robot name="robotiq_85_gripper" xmlns:xacro="http://ros.org/wiki/xacro">
     <xacro:include filename="$(find vector_description)/urdf/manipulation/robotiq/robotiq_85_gripper.transmission.xacro" />
-    <property name="pi" value="3.14159"/>
+    <xacro:property name="pi" value="3.14159"/>
     <xacro:macro name="robotiq_85_gripper" params="prefix parent *origin">
         <joint name="${prefix}robotiq_85_base_joint" type="fixed">

File: vector_common/vector_description/urdf/sensors/pan_tilt_kinect_one.urdf.xacro (robot description, xacro)
@@ -23,5 +23,5 @@
 <robot name="pan_tilt_kinect_one" xmlns:xacro="http://ros.org/wiki/xacro">
 	<xacro:include filename="$(find vector_description)/urdf/sensors/kinect_one_sensor.urdf.xacro"/>
-    <property name="M_PI" value="3.14159"/>
+    <xacro:property name="M_PI" value="3.14159"/>
     <xacro:macro name="pan_tilt_kinect_one" params="rgbd_prefix parent *origin">
         <joint name="pan_base_joint" type="fixed">
